File: placa_electronica/pcb_ojo_de_van_gogh/pcb_ojo_de_van_gogh.kicad_pcb (KiCad board)
At the start: 2 copper layers, 15 parts, among them U1 Ultrasonico, U2 Switch-4-posiciones, U3 Buzzer, U4 HC-05, U5 Buzzer, U6 PiZeroW

Commit message: 3D-Huellas
Parts:
- removed U1: Ultrasonico, VibradorPCB:Ultrasonico
